File: hrbl-shield/dev_files/grbl_shield.sch (EAGLE design)
At the start: 16 parts, among them Q1 ARDUINOR3-NOIOREF-NOTEXT

Commit message: moved in dev and shield update
Parts:
- removed C4: 100nF, fab:CAP-UNPOLARIZEDFAB
- removed SPINDLE: (no value), pinhead:PINHD-1X4
Connections:
- net ABORT: no longer C4.1
- net GND: no longer C4.2
- net SPINDLE_COM: no longer SPINDLE.2
- net SPINDLE_PWM: no longer SPINDLE.4
- net SPINDLE_RUN: no longer SPINDLE.1
Other:
- note added: "ACM"
- note added: "Red"
- note added: "acm grønn"
- note added: "blå"
- note added: "brun"
- note added: "dmc Grå"
- note added: "for lilla"
- note added: "grå"
- note added: "grønn"
- note added: "gul"
- note added: "lilla"
- note added: "orange"
- note added: "replaced with optocouplers"
- note added: "rød"
- note added: "vi blå"
- note removed: "Blå"
- note removed: "Brun"
- note removed: "Grå"
- note removed: "Grønn"
- note removed: "Gul"
- note removed: "Lila"
- note removed: "Orange"
- note removed: "Rød"
- note removed: "spindle on"
- moved on the sheet: IHSS60, RIBBON_X
