File: humphrey-large-format-cnc/new-dev-files/humphrey v2/newtone_settings/grbl_shield_hector.sch (EAGLE design)
At the start: 15 parts, among them Q1 ARDUINOR3-NOIOREF-NOTEXT

Commit message: fab14
Parts:
- added RIBBON_XOLD, RIBBON_XZ, RIBBON_Y1, RIBBON_Y1_Y2, RIBBON_Y2, RIBBON_Z, S1, S2: (no value), pinhead:PINHD-1X8
- renumbered RIBBON_X1 to RIBBON_X1NOTUSED
Connections:
- net DIR_X renamed DIR+X
- net STEP_Y renamed PUL+Y
- net STEP_Z renamed PUL+Z
- new net 36V+: S1.7, S1.8
- new net 36V_GND: S1.2, S1.3, S1.4, S1.5, S1.6
- new net ARD_GND: S2.2
- new net N$6: RIBBON_X.5, RIBBON_X.7, RIBBON_Z.5, RIBBON_Z.7
- new net PUL+X: Q1.D2
- new net SENS+: S2.7
- new net SENS-: S2.5
- new net SIG-X_Z: S2.4
- new net SIG-_Y1_Y2: S2.3
- net ABORT: now also RIBBON_XOLD.5; no longer RIBBON_X.5
- net DC+: now also RIBBON_X.3, RIBBON_X1NOTUSED.1, RIBBON_XZ.3, RIBBON_Y1.3, RIBBON_Y1_Y2.3, RIBBON_Y2.3, RIBBON_Z.3, S2.8; no longer RIBBON_X1NOTUSED.2
- net DIR: now also RIBBON_XOLD.3; no longer RIBBON_X.3
- net DIR+: now also RIBBON_X.6, RIBBON_XZ.6, RIBBON_Y1.6, RIBBON_Y1_Y2.6, RIBBON_Y2.6, RIBBON_Z.6
- net DIR-: now also RIBBON_XZ.5, RIBBON_Y1_Y2.5
- net GND: now also RIBBON_X.4, RIBBON_X1NOTUSED.2, RIBBON_XOLD.2, RIBBON_XZ.4, RIBBON_Y1.4, RIBBON_Y1_Y2.4, RIBBON_Y2.4, RIBBON_Z.4, S2.6; no longer RIBBON_X.2, RIBBON_X1NOTUSED.1
- net LIMIT_X: now also RIBBON_XOLD.8; no longer RIBBON_X.8
- net PUL+: now also RIBBON_X.8, RIBBON_XZ.8, RIBBON_Y1.8, RIBBON_Y1_Y2.8, RIBBON_Y2.8, RIBBON_Z.8
- net PUL-: now also RIBBON_XZ.7, RIBBON_Y1.5, RIBBON_Y1.7, RIBBON_Y1_Y2.7, RIBBON_Y2.5, RIBBON_Y2.7
- net STEPPER_ENABLE: now also RIBBON_XOLD.4; no longer RIBBON_X.4
- net STEP_X: now also RIBBON_XOLD.1; no longer Q1.D2, RIBBON_X.1
- net VCC_36V+: now also RIBBON_XOLD.6; no longer RIBBON_X.6
- net VCC_GND: now also RIBBON_XOLD.7; no longer RIBBON_X.7
Other:
- note added: "DIR-"
- note added: "SIG-_X_Z"
- note added: "SIG-_Y1_Y2"
- note added: "SOCKERBIT"
- note added: "skip"
- moved on the sheet: RIBBON_X
