File: hrbl-shield/dev_files/test_pos/test_pos.kicad_pcb (KiCad board)
At the start: 2 copper layers, 9.7 x 10.9 mm, 5 parts

Commit message: more jlcpcb testing
Parts:
- removed C2: 10Fu, Capacitor_SMD:C_1206_3216Metric
- removed D1: LED, LED_THT:LED_D5.0mm
- removed R2: 1000, Resistor_SMD:R_1206_3216Metric
- R1: moved to B.Cu
- moved R1 24.3 mm to (40.1, 31.9)
- moved C1 2.44 mm to (17.3, 15.7)
Routing:
- net Net-(C1-Pad2): track 18.1 -> 32.8 mm, vias 0 -> 1
- net +5V: track 18.6 -> 30.2 mm, vias 0 -> 1
Other:
- board size 9.7 x 10.9 mm -> 32.1 x 24.4 mm
