File: hrbl-shield/dev_files/test_pos/test_pos.sch (KiCad schematic (older format))
At the start: 5 parts

Commit message: more jlcpcb testing
Parts:
- removed C2: 10Fu, Capacitor_SMD:C_1206_3216Metric, symbol Device:C
- removed D1: LED, LED_THT:LED_D5.0mm, symbol Device:LED
- removed R2: 1000, Resistor_SMD:R_1206_3216Metric, symbol Device:R
- C1: LCSC Part #（optional） (none) -> C13585
- R1: LCSC Part #（optional） (none) -> C4410
Changed lines of the file:
@@
 EESchema Schematic File Version 4
+LIBS:test_pos-cache
 EELAYER 26 0
 EELAYER END
@@
 F 2 "Resistor_SMD:R_1206_3216Metric" V 3980 2250 50  0001 C CNN
 F 3 "~" H 4050 2250 50  0001 C CNN
+F 4 "C4410 " H 4050 2250 50  0001 C CNN "LCSC Part #（optional）"
 	1    4050 2250
 	1    0    0    -1
@@
 F 2 "Capacitor_SMD:C_1206_3216Metric" H 4488 2100 50  0001 C CNN
 F 3 "~" H 4450 2250 50  0001 C CNN
+F 4 "C13585 " H 4450 2250 50  0001 C CNN "LCSC Part #（optional）"
 	1    4450 2250
 	1    0    0    -1
@@
 Wire Wire Line
 	4250 2100 4450 2100
-$Comp
-L Device:R R2
-U 1 1 5E2E55F6
-P 5250 2200
-F 0 "R2" H 5320 2246 50  0000 L CNN
-F 1 "1000" H 5320 2155 50  0000 L CNN
-F 2 "Resistor_SMD:R_1206_3216Metric" V 5180 2200 50  0001 C CNN
-F 3 "~" H 5250 2200 50  0001 C CNN
-	1    5250 2200
-	1    0    0    -1
-$EndComp
-$Comp
-L Device:C C2
-U 1 1 5E2E55FD
-P 5650 2200
-F 0 "C2" H 5765 2246 50  0000 L CNN
-F 1 "10Fu" H 5765 2155 50  0000 L CNN
-F 2 "Capacitor_SMD:C_1206_3216Metric" H 5688 2050 50  0001 C CNN
-F 3 "~" H 5650 2200 50  0001 C CNN
-	1    5650 2200
-	1    0    0    -1
-$EndComp
-Wire Wire Line
-	5250 2350 5650 2350
-$Comp
-L power:GND #PWR0101
-U 1 1 5E2E5606
-P 5450 2400
-F 0 "#PWR0101" H 5450 2150 50  0001 C CNN
-F 1 "GND" H 5455 2227 50  0000 C CNN
-F 2 "" H 5450 2400 50  0001 C CNN
-F 3 "" H 5450 2400 50  0001 C CNN
-	1    5450 2400
-	1    0    0    -1
-$EndComp
-Wire Wire Line
-	5250 2050 4950 2050
-Wire Wire Line
-	4450 2050 4450 2100
-Connection ~ 5250 2050
-Connection ~ 4450 2100
-Wire Wire Line
-	5250 2050 5650 2050
-Wire Wire Line
-	4450 2400 4950 2400
-Wire Wire Line
-	5250 2400 5250 2350
-Connection ~ 4450 2400
-Connection ~ 5250 2350
-$Comp
-L Device:LED D1
-U 1 1 5E2E5726
-P 4950 2250
-F 0 "D1" V 4895 2328 50  0000 L CNN
-F 1 "LED" V 4986 2328 50  0000 L CNN
-F 2 "LED_THT:LED_D5.0mm" H 4950 2250 50  0001 C CNN
-F 3 "~" H 4950 2250 50  0001 C CNN
-	1    4950 2250
-	0    1    1    0
-$EndComp
-Connection ~ 4950 2400
-Wire Wire Line
-	4950 2400 5250 2400
-Wire Wire Line
-	4950 2100 4950 2050
-Connection ~ 4950 2050
-Wire Wire Line
-	4950 2050 4450 2050
 $EndSCHEMATC
